Commit message: init visualization package

File: models/primius.urdf (robot description, URDF)
Before this commit: robot primius, 2 links, 1 joints
Joints:
- joint base_link_wheel_front_right: type fixed -> continuous

Commit message: fix visualization

File: models/primius.urdf (robot description, URDF)
Before this commit: robot primius, 2 links, 1 joints
Joints:
- joint base_link_wheel_front_right: type continuous -> fixed
