Commit message: four wheel in rviz

File: models/xacro/color.xacro (robot description, xacro)
@@ -7,3 +7,6 @@
         <color rgba="1 1 1 1"/>
     </material>
+    <material name="black">
+        <color rgba="0 0 0 1"/>
+    </material>
 </robot>

File: models/xacro/primius.urdf.xacro (robot description, xacro)
@@ -24,6 +24,6 @@
                 <mesh filename="package://visualization/meshes/mecanum_wheel.stl" scale="0.01 0.01 0.01"/>
             </geometry>
-            <material name="white"/>
-            <origin xyz="0.0 0.0 0.0" rpy="${pi/2} 0.0 0.0"/>
+            <!-- <material name="black"/> -->
+            <origin xyz="0.0 0.0 0.0" rpy="0.0 0.0 ${pi/2}"/>
         </visual>
     </link>
@@ -31,5 +31,50 @@
         <parent link="base_link"/>
         <child link="wheel_front_right"/>
-        <origin xyz="0.18 0.12 -${wheel_radius}" rpy="0.0 0.0 0.0"/>
+        <origin xyz="0.105 0.073 0.0" rpy="0.0 0.0 0.0"/>
+        <axis xyz="0 1 0"/>
+    </joint>
+    <link name="wheel_back_right">
+        <visual>
+            <geometry>
+                <mesh filename="package://visualization/meshes/mecanum_wheel.stl" scale="0.01 0.01 0.01"/>
+            </geometry>
+            <!-- <material name="black"/> -->
+            <origin xyz="0.0 0.0 0.0" rpy="0.0 0.0 ${pi/2}"/>
+        </visual>
+    </link>
+    <joint name="base_link_wheel_back_right" type="continuous">
+        <parent link="base_link"/>
+        <child link="wheel_back_right"/>
+        <origin xyz="-0.105 0.073 0.0" rpy="0.0 0.0 0.0"/>
+        <axis xyz="0 1 0"/>
+    </joint>
+    <link name="wheel_front_left">
+        <visual>
+            <geometry>
+                <mesh filename="package://visualization/meshes/mecanum_wheel.stl" scale="0.01 0.01 0.01"/>
+            </geometry>
+            <!-- <material name="black"/> -->
+            <origin xyz="0.0 0.0 0.0" rpy="0.0 0.0 -${pi/2}"/>
+        </visual>
+    </link>
+    <joint name="base_link_wheel_front_left" type="continuous">
+        <parent link="base_link"/>
+        <child link="wheel_front_left"/>
+        <origin xyz="0.105 -0.073 0.0" rpy="0.0 0.0 0.0"/>
+        <axis xyz="0 1 0"/>
+    </joint>
+    <link name="wheel_back_left">
+        <visual>
+            <geometry>
+                <mesh filename="package://visualization/meshes/mecanum_wheel.stl" scale="0.01 0.01 0.01"/>
+            </geometry>
+            <!-- <material name="black"/> -->
+            <origin xyz="0.0 0.0 0.0" rpy="0.0 0.0 -${pi/2}"/>
+        </visual>
+    </link>
+    <joint name="base_link_wheel_back_left" type="continuous">
+        <parent link="base_link"/>
+        <child link="wheel_back_left"/>
+        <origin xyz="-0.105 -0.073 0.0" rpy="0.0 0.0 0.0"/>
         <axis xyz="0 1 0"/>
     </joint>
