Commit message: kinect

File: models/xacro/primius.urdf.xacro (robot description, xacro)
@@ -79,3 +79,18 @@
         <axis xyz="0 1 0"/>
     </joint>
+    <link name="kinect_camera">
+        <visual>
+            <geometry>
+                <mesh filename="package://visualization/meshes/kinect.stl"/>
+            </geometry>
+            <material name="black"/>
+            <origin xyz="0.0 0.0 0.0" rpy="0.0 0.0 -${pi/2}"/>
+        </visual>
+    </link>
+    <joint name="base_link_kinect_camera" type="fixed">
+        <parent link="base_link"/>
+        <child link="kinect_camera"/>
+        <origin xyz="${base_lenght/2} 0.0 0.075" rpy="0.0 0.0 0.0"/>
+        <axis xyz="0 1 0"/>
+    </joint>
 </robot>
